File: Kicad/CPLD.kicad_sch (KiCad schematic)
At the start: 30 parts, among them J2 Conn_01x06_Male, J3 Conn_01x05_Pin, J4 Conn_02x03_Odd_Even, U6 XC95144XL-TQ100, U7 AZ1117-3.3, X1 50MHz

Commit message: Update JLC BOM & CPL * Include IDE Header and jumper block * Replace JLC part numbers with in-stock items (except flash)
Parts:
- J2, J3: now left out of the parts list
- J4: LCSC # (none) -> C7501274
- X1: LCSC # C46327 -> C5203552
Changed lines of the file:
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@@
 		(unit 1)
 		(exclude_from_sim no)
-		(in_bom yes)
+		(in_bom no)
 		(on_board yes)
 		(dnp no)
@@
 			)
 		)
-		(property "LCSC #" "C46327"
+		(property "LCSC #" "C5203552"
 			(at 107.95 140.97 0)
 			(effects
@@
 			)
 		)
+		(property "LCSC #" "C7501274"
+			(at 270.51 73.66 0)
+			(effects
+				(font
+					(size 1.27 1.27)
+				)
+				(hide yes)
+			)
+		)
 		(pin "5"
 		)
@@
 		(unit 1)
 		(exclude_from_sim no)
-		(in_bom yes)
-		(on_board yes)
-		(dnp no)
+		(in_bom no)
+		(on_board yes)
+		(dnp no)

Commit message: Update BOM
Add Digikey Part links (including new part number for Flash)
Removed EOL flash part link from Mouser
Parts:
- AMIGA1: Digikey # (none) -> ED5764-64-ND
- C13, C17, C18, C19, C20, C22, C23, C24: Digikey # (none) -> 399-C0603C104K5RAC3121CT-ND
- C14, C15: Digikey # (none) -> 399-5152-1-ND
- C21: Digikey # (none) -> 1276-CL21A106KQFNNWECT-ND
- J4: Digikey # (none) -> 4-146262-1-ND
- R1, R11, R2, R3, R8: Digikey # (none) -> A126394CT-ND
- R12, R20: Digikey # (none) -> A130406CT-ND
- R18, R19, R6, R7, R9: Digikey # (none) -> 1712-CRG0603F33RCT-ND
- U6: Mouser # 217-5144XL-10TQG100C -> 217-5144XL-10TQG100I
- U7: Digikey # (none) -> AZ1117CR-3.3TRG1DICT-ND
- X1: Digikey # (none) -> XC1930CT-ND
