File: Kicad/IDE.kicad_sch (KiCad schematic)
At the start: 21 parts, among them J1 IDE, U1 SST39SF010, U4 74HCT245, U8 74HCT245, U9 74HCT245

Commit message: Update JLC BOM & CPL * Include IDE Header and jumper block * Replace JLC part numbers with in-stock items (except flash)
Parts:
- F1: LCSC # (none) -> C21714343
- J1: LCSC # (none) -> C9138
Changed lines of the file:
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@@
+			)
+		)
+		(property "LCSC #" "C21714343"
+			(at 266.7 68.58 0)
+			(effects
+				(font
+					(size 1.27 1.27)
+				)
+				(hide yes)
 			)
 		)
@@
 			(at 231.14 76.2 0)
 			(effects
+				(font
+					(size 1.27 1.27)
+				)
+				(hide yes)
+			)
+		)
+		(property "LCSC #" "C9138"
+			(at 231.14 76.2 0)
+			(effects

Commit message: Update BOM
Add Digikey Part links (including new part number for Flash)
Removed EOL flash part link from Mouser
Parts:
- C1, C16, C3, C4: Digikey # (none) -> 399-C0603C104K5RAC3121CT-ND
- C26: Digikey # (none) -> 399-T490A476M010ATE1K0CT-ND
- D1: Digikey # (none) -> 67-1549-1-ND
- F1: Digikey # (none) -> 18-1206L110/16WRCT-ND
- J1: Digikey # (none) -> 2057-BHR-40-VUA-ND
- R10, R15, R16, R17, R4, R5: Digikey # (none) -> A126394CT-ND
- R13, R14: Digikey # (none) -> 1712-CRG0603F33RCT-ND
- R21: Digikey # (none) -> A130406CT-ND
- U1: Digikey # (none) -> 150-SST39SF010A-70-4C-TU-ND; Mouser # 579-SST39010A554CWHE -> (none)
- U4, U8, U9: Digikey # (none) -> 296-8404-1-ND
