File: Kicad/RAM.kicad_sch (KiCad schematic)
At the start: 13 parts, among them U2 74LVC245, U3 74LVC245, U5 W9812G6KH-6

Commit message: Update JLC BOM & CPL * Include IDE Header and jumper block * Replace JLC part numbers with in-stock items (except flash)
Parts:
- U5: LCSC # C367430 -> C62379
Changed lines of the file:
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@@
 			)
 		)
-		(property "LCSC #" "C367430"
+		(property "LCSC #" "C62379"
 			(at 240.03 89.535 0)
 			(effects
@@
 			)
 		)
-		(property "LCSC #" "C367430"
+		(property "LCSC #" "C62379"
 			(at 144.78 82.55 0)
 			(effects

Commit message: Update BOM
Add Digikey Part links (including new part number for Flash)
Removed EOL flash part link from Mouser
Parts:
- C10, C11, C12, C5, C6, C7, C8, C9: Digikey # (none) -> 399-C0603C104K5RAC3121CT-ND
- C25: Digikey # (none) -> 1276-CL21A106KQFNNWECT-ND
- U2, U3: Digikey # (none) -> 296-1233-1-ND
- U5: Digikey # (none) -> W9812G6KH-6-ND
